File: Kicad/3Channel-PiezoAmp/3Channel-PiezoAmp.sch (KiCad schematic (older format))
At the start: 5 parts

Commit message: finished schematics
Parts:
- added BT1: Battery, symbol Device:Battery
- added C1: 10uF, symbol Device:CP_Small
- added C10, C11, C12, C13, C8, C9: 1uF, symbol Device:CP_Small
- added C14: 100uF, symbol Device:C
- added C15: 10pF, symbol Device:C_Small
- added C16: 220uF, symbol Device:C
- added C17: 10nF, symbol Device:CP_Small
- added C2, C3, C4: 100nF, symbol Device:C_Small
- added C5, C6, C7: 1nF, symbol Device:C_Small
- added D1, D2, D3, D4, D5, D6: 1N4148, symbol Device:D
- added J1: InputJack1, symbol Connector:AudioJack3
- added J2: InputJack2, symbol Connector:AudioJack3
- added J3: InputJack3, symbol Connector:AudioJack3
- added J4: OutputJack1, symbol Connector:AudioJack3
- added J5: DC_Jack_SW_inv, symbol Connector:Barrel_Jack_Switch
- added LED1: LED1, symbol Device:LED
- added LED2: LED2, symbol Device:LED
- added LED3: LED3, symbol Device:LED
- added R1, R10, R11, R12, R2, R9: 10k, symbol Device:R
- added R13: 10, symbol Device:R
- added R14, R15, R16, R6, R7, R8: 1k, symbol Device:R
- added R3, R4, R5: 2.2M, symbol Device:R
- added RV1: Pot1, symbol Device:R_POT
- added RV2: Pot2, symbol Device:R_POT
- added RV3: Pot3, symbol Device:R_POT
- gave numbers to parts that had none: 1
Connections:
- net at U1.1: now also C7.1, R5.1, R8.2
- net at U1.2 (-): now also C4.1, C7.2, R5.2
- net 4.5V: now reaches U1.3 (+)
- net 4.5V: now also U1.10 (+), U1.12 (+), U1.5 (+), C1.1, R1.2, R2.1
- net at U1.6 (-): now also C15.2, R10.1, R11.1, R12.2, R9.1
- net at U1.7: now also C15.1, C17.1, R12.1
- net at U1.8: now also C6.1, R4.1, R7.2
- net at U1.9 (-): now also C3.1, C6.2, R4.2
- net at U1.13 (-): now also C2.1, C5.2, R3.2
- net at U1.14: now also C5.1, R3.1, R6.2
- net GND: now reaches U1.11 (V-)
- net GND: now also C1.2, C16.2, D2.2 (A), D4.2 (A), D6.2 (A), J1.S, J2.S, J3.S, J4.S, J5.1, R14.1, R15.1, R16.1, R2.2, RV1.3, RV2.3, RV3.3
- net +9V: now reaches U1.4 (V+)
- net +9V: now also D1.1 (K), D3.1 (K), D5.1 (K), J5.2, LED1.2 (A), LED2.2 (A), LED3.2 (A), R1.1, R13.1
- new net: C16.1, R13.2
- new net: C2.2, D1.2 (A), D2.1 (K), J1.T
- new net: C8.1, R6.1
- new net: C8.2, RV1.1
- new net: C11.1, RV1.2
- new net: C11.2, R9.2
- new net: C17.2, J4.T
- new net: C9.1, R7.1
- new net: C9.2, RV2.1
- new net: C12.1, RV2.2
- new net: C12.2, R10.2
- new net: C3.2, D3.2 (A), D4.1 (K), J2.T
- new net: C10.1, R8.1
- new net: C10.2, RV3.1
- new net: C13.1, RV3.2
- new net: C13.2, R11.2
- new net: C4.2, D5.2 (A), D6.1 (K), J3.T
- new net: LED1.1 (K), R14.2
- new net: LED3.1 (K), R16.2
- new net: LED2.1 (K), R15.2
- new net BatPlus: BT1.1 (+), C14.1, J5.3
- new net GNDswitch: BT1.2 (-), C14.2, J1.R, J2.R, J3.R
Other:
- note added: "Experimental\n"
- moved on the sheet: U1A, U1B, U1C, U1D, U1E
