File: Kicad/3Channel-PiezoAmp/3Channel-PiezoAmp.sch (KiCad schematic (older format))
At the start: 52 parts, among them J1 InputJack1, J2 InputJack2, J3 InputJack3, J4 OutputJack1, J5 DC_Jack_SW_inv, U1 TL074

Commit message: starting wiht 1chan
Parts:
- added Q1, Q2, Q3: BC547, Package_TO_SOT_SMD:SOT-23_Handsoldering, symbol Transistor_BJT:BC547
- added R17, R18, R19: 4.7k, Resistor_SMD:R_1206_3216Metric_Pad1.30x1.75mm_HandSolder, symbol Device:R
- C15: value 10pF -> 100pF
- C17: value 10nF -> 10uF
- J1, J2, J3, J4: footprint Connector_Audio:Jack_3.5mm_PJ320D_Horizontal -> 3Channel-PiezoAmp:Jack_3.5mm_dusjagr_Horizontal
- RV1, RV2, RV3: footprint Potentiometer_THT:Potentiometer_Alps_RK09K_Single_Vertical -> 3Channel-PiezoAmp:RD901F-ALPHA-3D
Connections:
- net labels added: Sig1, Sig2, Sig3
- wire segments 160 -> 187
Other:
- moved on the sheet: LED1, LED2, LED3, R14, R15, R16, U1E
