File: Kicad/3Channel-PiezoAmp/_autosave-3Channel-PiezoAmp.kicad_pcb (KiCad board)
At the start: 2 copper layers, 91.5 x 53 mm, 49 parts, among them J1 InputJack1, J2 InputJack2, J3 InputJack3, J4 OutputJack1, U1 TL074

Commit message: first PCB v01
Routing:
- net +9V: track 231.7 -> 240.5 mm, vias 4 -> 3
Changed lines of the file:
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@@
     (thickness 1.6)
     (drawings 6)
-    (tracks 360)
+    (tracks 358)
     (zones 0)
     (modules 49)
@@
     (visible_elements FFFFFF7F)
     (pcbplotparams
-      (layerselection 0x010fc_ffffffff)
+      (layerselection 0x01000_ffffffff)
       (usegerberextensions false)
       (usegerberattributes true)
@@
       (padsonsilk false)
       (subtractmaskfromsilk false)
-      (outputformat 1)
+      (outputformat 4)
       (mirror false)
-      (drillshape 0)
+      (drillshape 1)
       (scaleselection 1)
       (outputdirectory ""))
@@
   (via (at 81.28 68.58) (size 1.5) (drill 0.8) (layers F.Cu B.Cu) (net 28))
   (segment (start 81.28 66.0035) (end 81.28 68.58) (width 0.8) (layer B.Cu) (net 28))
-  (segment (start 44.704 100.584) (end 47.244 103.124) (width 0.8) (layer F.Cu) (net 28))
-  (segment (start 47.244 103.124) (end 59.436 103.124) (width 0.8) (layer F.Cu) (net 28))
-  (segment (start 59.436 103.124) (end 60.96 101.6) (width 0.8) (layer F.Cu) (net 28))
-  (via (at 60.96 101.6) (size 1.5) (drill 0.8) (layers F.Cu B.Cu) (net 28))
-  (segment (start 60.732 101.372) (end 60.96 101.6) (width 0.8) (layer B.Cu) (net 28))
-  (segment (start 60.732 96.266) (end 60.732 101.372) (width 0.8) (layer B.Cu) (net 28))
   (segment (start 45.212 84.328) (end 44.704 84.836) (width 0.8) (layer F.Cu) (net 28))
   (segment (start 54.864 84.328) (end 45.212 84.328) (width 0.4) (layer F.Cu) (net 28))
-  (segment (start 44.704 84.836) (end 44.704 100.584) (width 0.8) (layer F.Cu) (net 28))
   (segment (start 44.704 81.28) (end 44.704 84.836) (width 0.8) (layer F.Cu) (net 28))
   (segment (start 87.361989 84.328) (end 118.364 84.328) (width 0.4) (layer F.Cu) (net 28))
@@
   (segment (start 54.864 84.328) (end 58.928 84.328) (width 0.4) (layer F.Cu) (net 28))
   (segment (start 87.361989 84.328) (end 86.36 84.328) (width 0.4) (layer F.Cu) (net 28))
+  (segment (start 61.976 103.124) (end 67.31 97.79) (width 0.8) (layer F.Cu) (net 28))
+  (segment (start 67.31 97.79) (end 73.66 97.79) (width 0.8) (layer F.Cu) (net 28))
+  (segment (start 47.244 103.124) (end 61.976 103.124) (width 0.8) (layer F.Cu) (net 28))
+  (segment (start 44.704 100.584) (end 47.244 103.124) (width 0.8) (layer F.Cu) (net 28))
+  (segment (start 44.704 84.836) (end 44.704 100.584) (width 0.8) (layer F.Cu) (net 28))
   (segment (start 55.906 71.628) (end 55.906 74.65) (width 0.4) (layer F.Cu) (net 29))
   (segment (start 54.61 75.946) (end 54.61 78.985) (width 0.4) (layer F.Cu) (net 29))
