File: Kicad/3Channel-PiezoAmp/_autosave-3Channel-PiezoAmp.sch (KiCad schematic (older format))
At the start: 52 parts, among them J1 InputJack1, J2 InputJack2, J3 InputJack3, J4 OutputJack1, J5 DC_Jack_SW_inv, U1 TL074

Commit message: first PCB v01
Parts:
- J1, J2, J3, J4: footprint Connector_Audio:Jack_3.5mm_PJ320D_Horizontal -> 3Channel-PiezoAmp:Jack_3.5mm_dusjagr_Horizontal
Changed lines of the file:
@@
 F 0 "J1" H 1032 3275 50  0000 C CNN
 F 1 "InputJack1" H 1032 3184 50  0000 C CNN
-F 2 "Connector_Audio:Jack_3.5mm_PJ320D_Horizontal" H 1050 2950 50  0001 C CNN
+F 2 "3Channel-PiezoAmp:Jack_3.5mm_dusjagr_Horizontal" H 1050 2950 50  0001 C CNN
 F 3 "~" H 1050 2950 50  0001 C CNN
 	1    1050 2950
@@
 F 0 "J4" H 9770 1983 50  0000 R CNN
 F 1 "OutputJack1" H 9770 2074 50  0000 R CNN
-F 2 "Connector_Audio:Jack_3.5mm_PJ320D_Horizontal" H 10050 2050 50  0001 C CNN
+F 2 "3Channel-PiezoAmp:Jack_3.5mm_dusjagr_Horizontal" H 10050 2050 50  0001 C CNN
 F 3 "~" H 10050 2050 50  0001 C CNN
 	1    10050 2050
@@
 F 0 "J2" H 1032 5425 50  0000 C CNN
 F 1 "InputJack2" H 1032 5334 50  0000 C CNN
-F 2 "Connector_Audio:Jack_3.5mm_PJ320D_Horizontal" H 1050 5100 50  0001 C CNN
+F 2 "3Channel-PiezoAmp:Jack_3.5mm_dusjagr_Horizontal" H 1050 5100 50  0001 C CNN
 F 3 "~" H 1050 5100 50  0001 C CNN
 	1    1050 5100
@@
 F 0 "J3" H 1032 7175 50  0000 C CNN
 F 1 "InputJack3" H 1032 7084 50  0000 C CNN
-F 2 "Connector_Audio:Jack_3.5mm_PJ320D_Horizontal" H 1050 6850 50  0001 C CNN
+F 2 "3Channel-PiezoAmp:Jack_3.5mm_dusjagr_Horizontal" H 1050 6850 50  0001 C CNN
 F 3 "~" H 1050 6850 50  0001 C CNN
 	1    1050 6850
