File: Kicad/3Channel-PiezoAmp/3Channel-PiezoAmp.kicad_pcb (KiCad board)
At the start: 2 copper layers, 91.5 x 53 mm, 49 parts, among them J1 InputJack1, J2 InputJack2, J3 InputJack3, J4 OutputJack1, U1 TL074

Commit message: starting wiht 1chan
Parts:
- added Q1: BC547, Package_TO_SOT_SMD:SOT-23_Handsoldering, F.Cu at (48.3, 72.1)
- added Q2: BC547, Package_TO_SOT_SMD:SOT-23_Handsoldering, F.Cu at (97.0, 72.6)
- added Q3: BC547, Package_TO_SOT_SMD:SOT-23_Handsoldering, F.Cu at (110.7, 72.1)
- added R17: 4.7k, Resistor_SMD:R_1206_3216Metric_Pad1.30x1.75mm_HandSolder, F.Cu at (46.7, 84.3)
- added R18: 4.7k, Resistor_SMD:R_1206_3216Metric_Pad1.30x1.75mm_HandSolder, F.Cu at (95.5, 84.3)
- added R19: 4.7k, Resistor_SMD:R_1206_3216Metric_Pad1.30x1.75mm_HandSolder, F.Cu at (109.2, 84.3)
- C1, C14: footprint Capacitor_SMD:C_1210_3225Metric_Pad1.33x2.70mm_HandSolder -> Capacitor_THT:CP_Radial_D5.0mm_P2.50mm; moved to F.Cu
- C15: value 10pF -> 100pF
- C17: value 10nF -> 10uF
- moved R15 3.05 mm to (89.4, 71.6), turned to 180 degrees
- moved C1 1.52 mm to (55.9, 101.1)
- moved C14 1.02 mm to (68.6, 98.0)
Connections:
- net Net-(C11-Pad1) renamed Sig1
- net Net-(C12-Pad1) renamed Sig2
- net Net-(C13-Pad1) renamed Sig3
- R14 pad 1: GND -> Net-(Q1-Pad1)
- R15 pad 1: GND -> Net-(Q2-Pad1)
- R16 pad 1: GND -> Net-(Q3-Pad1)
Routing:
- net Net-(Q2-Pad2): track 0.00 -> 15.6 mm
- net GND: track 257.6 -> 245.4 mm
- net Sig3: track 22.2 -> 33.6 mm
- net Net-(Q3-Pad2): track 0.00 -> 9.70 mm
- net Net-(Q1-Pad2): track 0.00 -> 9.70 mm
- net Sig1: track 56.0 -> 65.4 mm
- net Net-(Q1-Pad1): track 0.00 -> 9.32 mm
- net +9V: track 231.7 -> 240.6 mm, vias 4 -> 3
- net Net-(Q3-Pad1): track 0.00 -> 8.70 mm
- net Net-(Q2-Pad1): track 0.00 -> 4.60 mm
- net Sig2: track 17.8 -> 19.3 mm
- net Net-(C7-Pad1): track 69.0 -> 67.8 mm
- net GNDswitch: track 133.7 -> 134.6 mm
