File: Kicad/1Channel-PiezoAmp/1Channel-PiezoAmp.sch (KiCad schematic (older format))
At the start: 28 parts, among them J1 InputJack1, J2 OutputJack1, J3 DC_Jack_SW_inv, Q1 BC547, U1 TL072

Commit message: starting wiht 1chan
Connections:
- net at C7.2, R7.1, R8.2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: no longer C5.2, R7.2
- new net: C5.2, R7.2
Changed lines of the file:
@@
 $EndComp
-Wire Wire Line
-	5700 2550 6000 2550
-Connection ~ 6000 2550
 Wire Wire Line
 	6000 2550 6300 2550
@@
 Wire Wire Line
 	5700 2550 5550 2550
-Connection ~ 5700 2550
 Wire Wire Line
 	5150 2550 5200 2550
